File: c1kshim.kicad_pcb (KiCad board)
At the start: 2 copper layers, 61 x 25 mm, 6 parts, among them J1 Conn_01x14, J11 Conn_02x20_Odd_Even, J12 Conn_02x06_Odd_Even, J2 Conn_01x14, J3 Conn_01x03, J4 Conn_01x02

Commit message: Correct comments
Other:
- board text added: "Note - this is a redo of the ck1shim from Sytse van Slooten. The holes should be in the exact right spots, but the tracks are somewhat different."
- board text removed: "Note - this is a redo of the ck1shim from sytse. The holes should be in the exact right spots, but the tracks are somewhat different."

Commit message: Add silk comment
Other:
- board text added: "c1kshim v1 Falco redo http://pdp2011.sytse.net/"

Commit message: Move to KiCad 6
Other:
- net class Default removed
